File: LEOS-stack-template.kicad_sch (KiCad schematic)
At the start: 23 parts, among them J1 MicroFit_1x4, J2 MicroFit_1x4, U1 MCP2562FD, U2 MCP2518FD, Y1 40 MHz

Commit message: Redesigned Rev 2 fixing 0603 cap size and layout
Parts:
- removed H1, H2, H3, H4: M3 Standoff Mount, MountingHole:MountingHole_3.2mm_M3, symbol Mechanical:MountingHole
- removed NT1: NetTie_2, Jumper:SolderJumper-2_P1.3mm_Bridged_RoundedPad1.0x1.5mm, symbol Device:NetTie_2
- added JP1: AGND Tie, Jumper:SolderJumper-2_P1.3mm_Bridged_RoundedPad1.0x1.5mm, symbol Jumper:SolderJumper_2_Bridged
- C1, C10, C11, C2, C3, C4, C5, C6, C7, C8, C9: footprint Capacitor_SMD:C_0201_0603Metric -> Capacitor_SMD:C_0603_1608Metric
- Y1: MPN (none) -> C13738
Connections:
- net GND: now also JP1.1 (A)
- net at A1.33 (AGND): now also JP1.2 (B)
Other:
- note removed: "Hardware"

Commit message: New redesign featuring updated components, new sheets, better routing, and 100% 3D View
Parts:
- removed C1, C2: 12pF, Capacitor_SMD:C_0603_1608Metric, symbol Device:C
- removed C3, C5, C7, C9: 0.1uF, Capacitor_SMD:C_0603_1608Metric, symbol Device:C
- removed C4, C6: 1uF, Capacitor_SMD:C_0603_1608Metric, symbol Device:C
- removed C8: 47uF, Capacitor_SMD:C_0603_1608Metric, symbol Device:C
- removed J1, J2: MicroFit_1x4, Connector_Molex:Molex_Micro-Fit_3.0_43650-0410_1x04-1MP_P3.00mm_Horizontal_PnP, symbol Connector:Conn_01x04_Pin
- removed JP1: AGND Tie, Jumper:SolderJumper-2_P1.3mm_Bridged_RoundedPad1.0x1.5mm, symbol Jumper:SolderJumper_2_Bridged
- removed R1: 120R, Resistor_THT:R_Axial_DIN0207_L6.3mm_D2.5mm_P7.62mm_Horizontal, symbol Device:R
- removed U1: MCP2562FD, Package_SO:SOIC-8_3.9x4.9mm_P1.27mm, symbol LEOS:MCP2562FD
- removed U2: MCP2518FD, Package_SO:SOIC-14_3.9x8.7mm_P1.27mm, symbol LEOS:MCP2518FD
- removed Y1: 40 MHz, Crystal:Crystal_SMD_3225-4Pin_3.2x2.5mm_HandSoldering, symbol Device:Crystal_GND24
- A1: value RaspberryPi_Pico -> RaspberryPi Pico; Digikey (none) -> 1778-PIM724-ND; MPN (none) -> PIM724; Manufacturer (none) -> Pimoroni
- C10: value 0.1uF -> 0.1u; Digikey (none) -> 490-5798-1-ND; MPN (none) -> CL10B104KB8NNNL; Manufacturer (none) -> Samsung Electro-Mechanics
- C11: value 10uF -> 10u; footprint Capacitor_SMD:C_0603_1608Metric -> Capacitor_SMD:C_0805_2012Metric; Digikey (none) -> 1276-2872-1-ND; MPN (none) -> CL21B106KOQNNNE; Manufacturer (none) -> Samsung Electro-Mechanics
Connections:
- net ADC0: no longer names the net of A1.31 (GPIO26_ADC0)
- net ADC1: no longer names the net of A1.32 (GPIO27_ADC1)
- net ADC2: no longer names the net of A1.34 (GPIO28_ADC2)
- net CAN_CS renamed CANbus/CS
- net CAN_INT renamed CANbus/INT
- net CAN_MISO renamed CANbus/MISO
- net CAN_MOSI renamed CANbus/MOSI
- net CAN_SCK renamed CANbus/SCK
- net GP10: no longer names the net of A1.14 (GPIO10)
- net GP11: no longer names the net of A1.15 (GPIO11)
- net GP12: no longer names the net of A1.16 (GPIO12)
- net GP13: no longer names the net of A1.17 (GPIO13)
- net GP14: no longer names the net of A1.19 (GPIO14)
- net GP15: no longer names the net of A1.20 (GPIO15)
- net GP16: no longer names the net of A1.21 (GPIO16)
- net GP17: no longer names the net of A1.22 (GPIO17)
- net GP18: no longer names the net of A1.24 (GPIO18)
- net GP19: no longer names the net of A1.25 (GPIO19)
- net GP20: no longer names the net of A1.26 (GPIO20)
- net GP21: no longer names the net of A1.27 (GPIO21)
- net GP22: no longer names the net of A1.29 (GPIO22)
- net GP7: no longer names the net of A1.10 (GPIO7)
- net I2C0_SCL: no longer names the net of A1.12 (GPIO9)
- net I2C0_SDA: no longer names the net of A1.11 (GPIO8)
- net RUN: no longer names the net of A1.30 (RUN)
- net UART0_RX: no longer names the net of A1.2 (GPIO1)
- net UART0_TX: no longer names the net of A1.1 (GPIO0)
- no-connect marks 6 -> 26
Other:
- added sheet CANbus (canbus.kicad_sch)
- added sheet Connectors (connectors.kicad_sch)
- note added: "AGND is internally connected."
- note added: "I2C0"
- note added: "SCK MOSI MISO CS"
- note added: "SDA SCL"
- note added: "SPI0"
- note added: "SPI1"
- note added: "Since CANbus is very high throughput, avoid using SPI0 for any other devices."
- note added: "TX RX"
- note added: "UART0"
- note removed: "BUS IN"
- note removed: "BUS OUT"
- note removed: "Bus Terminals"
- note removed: "CANBUS Comms"
- note removed: "Termination Resistor"
- title: LEOS Stack - Microcontroller & Connectivity -> LEOS Microcontroller
- moved on the sheet: A1, C10, C11

Commit message: Improved via placement, added LCSC part numbers.
Parts:
- C10: LCSC (none) -> C913912
- C11: LCSC (none) -> C95841
Changed lines of the file:
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@@
+	)
+	(no_connect
+		(at 170.18 106.68)
+	)
+	(no_connect
+		(at 170.18 99.06)
+	)
+	(no_connect
+		(at 170.18 93.98)
+	)
+	(no_connect
+		(at 124.46 83.82)
+	)
+	(no_connect
+		(at 124.46 109.22)
+	)
+	(no_connect
+		(at 124.46 106.68)
+	)
+	(no_connect
+		(at 170.18 119.38)
+	)
+	(no_connect
+		(at 170.18 127)
+	)
+	(no_connect
+		(at 124.46 116.84)
+	)
+	(no_connect
+		(at 170.18 91.44)
+	)
+	(no_connect
+		(at 124.46 124.46)
+	)
+	(no_connect
+		(at 124.46 91.44)
 	)
 	(no_connect
@@
 	)
 	(no_connect
-		(at 170.18 106.68)
-	)
-	(no_connect
-		(at 170.18 99.06)
-	)
-	(no_connect
-		(at 170.18 93.98)
-	)
-	(no_connect
-		(at 124.46 83.82)
-	)
-	(no_connect
-		(at 124.46 109.22)
-	)
-	(no_connect
-		(at 124.46 106.68)
-	)
-	(no_connect
-		(at 170.18 119.38)
-	)
-	(no_connect
-		(at 170.18 127)
-	)
-	(no_connect
-		(at 124.46 116.84)
-	)
-	(no_connect
-		(at 170.18 91.44)
-	)
-	(no_connect
-		(at 124.46 91.44)
-	)
-	(no_connect
 		(at 124.46 119.38)
 	)
@@
 	(no_connect
 		(at 170.18 96.52)
-	)
-	(no_connect
-		(at 124.46 124.46)
 	)
 	(no_connect
@@
 			)
 		)
+		(property "LCSC" "C95841"
+			(at 161.29 60.96 0)
+			(effects
+				(font
+					(size 1.27 1.27)
+				)
+				(hide yes)
+			)
+		)
 		(pin "2"
 		)
@@
 			)
 		)
-		(property "LCSC" ""
+		(property "LCSC" "C913912"
 			(at 130.81 60.96 0)
 			(effects

Commit message: Update bad part num for 0.1u
Parts:
- C10: Digikey 490-5798-1-ND -> 1276-CL10B104KB8NNNLCT-ND
Changed lines of the file:
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@@
+			)
+		)
+		(property "Sim.Pins" ""
+			(at 147.32 104.14 0)
+			(effects
+				(font
+					(size 1.27 1.27)
+				)
+				(hide yes)
 			)
 		)
@@
 			)
 		)
+		(property "Sim.Pins" ""
+			(at 161.29 60.96 0)
+			(effects
+				(font
+					(size 1.27 1.27)
+				)
+				(hide yes)
+			)
+		)
 		(pin "2"
 		)
@@
 			)
 		)
-		(property "Digikey" "490-5798-1-ND"
+		(property "Digikey" "1276-CL10B104KB8NNNLCT-ND"
 			(at 130.81 60.96 0)
 			(effects
@@
 			(at 130.81 60.96 0)
 			(effects
+				(font
+					(size 1.27 1.27)
+				)
+				(hide yes)
+			)
+		)
+		(property "Sim.Pins" ""
+			(at 130.81 60.96 0)
+			(effects
