File: canbus.kicad_sch (KiCad schematic)
At the start: 12 parts, among them U1 MCP2562FD, U2 MCP2518FD, Y1 40 MHz

Commit message: Improved via placement, added LCSC part numbers.
Parts:
- C1, C2: LCSC (none) -> C1634
- C3, C5, C7: LCSC (none) -> C913912
- C4, C6: LCSC (none) -> C29936
- U1: LCSC (none) -> C511335
- U2: LCSC (none) -> C626758
- Y1: LCSC (none) -> C5357833
Changed lines of the file:
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@@
+			)
+		)
+		(property "LCSC" "C1634"
+			(at 154.94 68.58 0)
+			(effects
+				(font
+					(size 1.27 1.27)
+				)
+				(hide yes)
 			)
 		)
@@
 			)
 		)
-		(property "LCSC" ""
+		(property "LCSC" "C29936"
 			(at 99.06 48.26 0)
 			(effects
@@
 			)
 		)
-		(property "LCSC" ""
+		(property "LCSC" "C913912"
 			(at 91.44 48.26 0)
 			(effects
@@
 			)
 		)
-		(property "LCSC" ""
+		(property "LCSC" "C29936"
 			(at 80.01 48.26 0)
 			(effects
@@
 			)
 		)
-		(property "LCSC" ""
+		(property "LCSC" "C913912"
 			(at 127 48.26 0)
 			(effects
@@
 			)
 		)
+		(property "LCSC" "C1634"
+			(at 140.97 68.58 0)
+			(effects
+				(font
+					(size 1.27 1.27)
+				)
+				(hide yes)
+			)
+		)
 		(pin "1"
 		)
@@
 			)
 		)
-		(property "LCSC" ""
+		(property "LCSC" "C511335"
 			(at 107.95 67.31 0)
 			(effects
@@
 			)
 		)
-		(property "LCSC" ""
+		(property "LCSC" "C626758"
 			(at 66.04 71.12 0)
 			(effects
@@
 			)
 		)
+		(property "LCSC" "C5357833"
+			(at 148.59 64.77 0)
+			(effects
+				(font
+					(size 1.27 1.27)
+				)
+				(hide yes)
+			)
+		)
 		(pin "4"
 		)
@@
 			)
 		)
-		(property "LCSC" ""
+		(property "LCSC" "C913912"
 			(at 72.39 48.26 0)
 			(effects

Commit message: Update bad part num for 0.1u
Parts:
- C3, C5, C7: Digikey 490-5798-1-ND -> 1276-CL10B104KB8NNNLCT-ND
Changed lines of the file:
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@@
+			)
+		)
+		(property "Sim.Pins" ""
+			(at 154.94 68.58 0)
+			(effects
+				(font
+					(size 1.27 1.27)
+				)
+				(hide yes)
 			)
 		)
@@
 			)
 		)
+		(property "Sim.Pins" ""
+			(at 119.38 64.77 0)
+			(effects
+				(font
+					(size 1.27 1.27)
+				)
+				(hide yes)
+			)
+		)
 		(pin "1"
 		)
@@
 			)
 		)
+		(property "Sim.Pins" ""
+			(at 99.06 48.26 0)
+			(effects
+				(font
+					(size 1.27 1.27)
+				)
+				(hide yes)
+			)
+		)
 		(pin "2"
 		)
@@
 			)
 		)
-		(property "Digikey" "490-5798-1-ND"
+		(property "Digikey" "1276-CL10B104KB8NNNLCT-ND"
 			(at 91.44 48.26 0)
 			(effects
@@
 		)
 		(property "Manufacturer" "Samsung Electro-Mechanics"
+			(at 91.44 48.26 0)
+			(effects
+				(font
+					(size 1.27 1.27)
+				)
+				(hide yes)
+			)
+		)
+		(property "Sim.Pins" ""
 			(at 91.44 48.26 0)
 			(effects
@@
 			)
 		)
+		(property "Sim.Pins" ""
+			(at 121.92 66.04 0)
+			(effects
+				(font
+					(size 1.27 1.27)
+				)
+				(hide yes)
+			)
+		)
 		(pin "1"
 		)
@@
 			)
 		)
+		(property "Sim.Pins" ""
+			(at 80.01 48.26 0)
+			(effects
+				(font
+					(size 1.27 1.27)
+				)
+				(hide yes)
+			)
+		)
 		(pin "2"
 		)
@@
 			)
 		)
-		(property "Digikey" "490-5798-1-ND"
+		(property "Digikey" "1276-CL10B104KB8NNNLCT-ND"
 			(at 127 48.26 0)
 			(effects
@@
 		)
 		(property "Manufacturer" "Samsung Electro-Mechanics"
+			(at 127 48.26 0)
+			(effects
+				(font
+					(size 1.27 1.27)
+				)
+				(hide yes)
+			)
+		)
+		(property "Sim.Pins" ""
 			(at 127 48.26 0)
 			(effects
@@
 			)
 		)
+		(property "Sim.Pins" ""
+			(at 140.97 68.58 0)
+			(effects
+				(font
+					(size 1.27 1.27)
+				)
+				(hide yes)
+			)
+		)
 		(pin "1"
 		)
@@
 			)
 		)
+		(property "Sim.Pins" ""
+			(at 107.95 67.31 0)
+			(effects
+				(font
+					(size 1.27 1.27)
+				)
+				(hide yes)
+			)
+		)
 		(pin "9"
 		)
@@
 			)
 		)
+		(property "Sim.Pins" ""
+			(at 66.04 71.12 0)
+			(effects
+				(font
+					(size 1.27 1.27)
+				)
+				(hide yes)
+			)
+		)
 		(pin "12"
 		)
@@
 			)
 		)
+		(property "Sim.Pins" ""
+			(at 148.59 64.77 0)
+			(effects
+				(font
+					(size 1.27 1.27)
+				)
+				(hide yes)
+			)
+		)
 		(pin "4"
 		)
@@
 			)
 		)
-		(property "Digikey" "490-5798-1-ND"
+		(property "Digikey" "1276-CL10B104KB8NNNLCT-ND"
 			(at 72.39 48.26 0)
 			(effects
@@
 			(at 72.39 48.26 0)
 			(effects
+				(font
+					(size 1.27 1.27)
+				)
+				(hide yes)
+			)
+		)
+		(property "Sim.Pins" ""
+			(at 72.39 48.26 0)
+			(effects
