File: connectors.kicad_sch (KiCad schematic)
At the start: 7 parts, among them J1 MicroFit_1x4, J2 MicroFit_1x4

Commit message: Improved via placement, added LCSC part numbers.
Parts:
- C8, C9: LCSC (none) -> C29936
- J1, J2: LCSC (none) -> C563846
Changed lines of the file:
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@@
 			)
 		)
-		(property "LCSC" ""
+		(property "LCSC" "C29936"
 			(at 114.3 52.07 0)
 			(effects
@@
 			)
 		)
+		(property "LCSC" "C563846"
+			(at 85.09 50.8 0)
+			(effects
+				(font
+					(size 1.27 1.27)
+				)
+				(hide yes)
+			)
+		)
 		(pin "4"
 		)
@@
 			)
 		)
-		(property "LCSC" ""
+		(property "LCSC" "C29936"
 			(at 121.92 52.07 0)
 			(effects
@@
 			(at 85.09 73.66 0)
 			(effects
+				(font
+					(size 1.27 1.27)
+				)
+				(hide yes)
+			)
+		)
+		(property "LCSC" "C563846"
+			(at 85.09 73.66 0)
+			(effects
